File: usbasp 16MHz/usbasp 28P 16Mhz/usbasp16Mhz.sch (KiCad schematic (older format))
At the start: 5 parts, among them J1 Conn_01x06_Male, U1 ATmega328P-PU, Y1 16MHz

Commit message: initial commit
Parts:
- U1: symbol MCU_Microchip_ATmega:ATmega328P-PU -> usbasp16Mhz-rescue:ATmega328P-PU-MCU_Microchip_ATmega
Changed lines of the file:
@@
 $EndDescr
 $Comp
-L MCU_Microchip_ATmega:ATmega328P-PU U1
+L usbasp16Mhz-rescue:ATmega328P-PU-MCU_Microchip_ATmega U1
 U 1 1 5FC8D473
 P 4350 4150
