File: usbasp target/usbasp target.sch (KiCad schematic (older format))
At the start: 4 parts, among them J1 Conn_01x06_Male, U1 ATtiny13-20PU, U2 ATtiny2313V-10PU, U3 ATmega8-16PU

Commit message: new symbols
Parts:
- U1: symbol MCU_Microchip_ATtiny:ATtiny13-20PU -> usbasp-target-rescue:ATtiny13-20PU-MCU_Microchip_ATtiny
- U2: symbol MCU_Microchip_ATtiny:ATtiny2313V-10PU -> usbasp-target-rescue:ATtiny2313V-10PU-MCU_Microchip_ATtiny
- U3: symbol MCU_Microchip_ATmega:ATmega8-16PU -> usbasp-target-rescue:ATmega8-16PU-MCU_Microchip_ATmega
Changed lines of the file:
@@
 $EndDescr
 $Comp
-L MCU_Microchip_ATtiny:ATtiny13-20PU U1
+L usbasp-target-rescue:ATtiny13-20PU-MCU_Microchip_ATtiny U1
 U 1 1 5FA129F9
 P 4650 2500
@@
 $EndComp
 $Comp
-L MCU_Microchip_ATmega:ATmega8-16PU U3
+L usbasp-target-rescue:ATmega8-16PU-MCU_Microchip_ATmega U3
 U 1 1 5FA13926
 P 7150 3300
@@
 $EndComp
 $Comp
-L MCU_Microchip_ATtiny:ATtiny2313V-10PU U2
+L usbasp-target-rescue:ATtiny2313V-10PU-MCU_Microchip_ATtiny U2
 U 1 1 5FA14768
 P 4700 5400
